File: 04_sch/CAN_controller.kicad_sch (KiCad schematic)
At the start: 12 parts, among them U4 TJA1050, U5 MCP2515-I_SO, Y1 Crystal

Commit message: Fix tantalum capacitor & JLCPCB codes
Parts:
- C15, C17: value 0.1uF -> 100nF; LCSC (none) -> C49678
- C16: footprint Capacitor_Tantalum_SMD:CP_EIA-1608-08_AVX-J_Pad1.25x1.05mm_HandSolder -> Capacitor_Tantalum_SMD:CP_EIA-2012-12_Kemet-R_Pad1.30x1.05mm_HandSolder; LCSC (none) -> C201218
- C18, C19: LCSC (none) -> C157623
- R15: LCSC (none) -> C191101
- R16: LCSC (none) -> C966144
- U5: LCSC (none) -> C5250735
- Y1: LCSC (none) -> C252310
Changed lines of the file:
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@@
 			)
 		)
-		(property "Value" "0.1uF"
+		(property "Value" "100nF"
 			(at 133.3563 77.47 90)
 			(effects
@@
 			)
 		)
-		(property "LCSC" ""
+		(property "LCSC" "C49678"
 			(at 133.35 81.28 0)
 			(effects
@@
 			)
 		)
-		(property "LCSC" ""
+		(property "LCSC" "C157623"
 			(at 49.53 100.33 0)
 			(effects
@@
 			)
 		)
-		(property "Footprint" "Capacitor_Tantalum_SMD:CP_EIA-1608-08_AVX-J_Pad1.25x1.05mm_HandSolder"
+		(property "Footprint" "Capacitor_Tantalum_SMD:CP_EIA-2012-12_Kemet-R_Pad1.30x1.05mm_HandSolder"
 			(at 123.19 76.2 0)
 			(effects
@@
 			)
 		)
-		(property "LCSC" ""
+		(property "LCSC" "C201218"
 			(at 123.19 76.2 0)
 			(effects
@@
 			)
 		)
-		(property "Value" "0.1uF"
+		(property "Value" "100nF"
 			(at 133.3563 67.31 90)
 			(effects
@@
 			)
 		)
-		(property "LCSC" ""
+		(property "LCSC" "C49678"
 			(at 133.35 71.12 0)
 			(effects
@@
 			)
 		)
-		(property "LCSC" ""
+		(property "LCSC" "C191101"
 			(at 133.35 90.17 0)
 			(effects
@@
 			)
 		)
-		(property "LCSC" ""
+		(property "LCSC" "C5250735"
 			(at 107.95 107.95 0)
 			(effects
@@
 			)
 		)
-		(property "LCSC" ""
+		(property "LCSC" "C252310"
 			(at 55.88 105.41 0)
 			(effects
@@
 			)
 		)
-		(property "LCSC" ""
+		(property "LCSC" "C157623"
 			(at 49.53 110.49 0)
 			(effects
@@
 			)
 		)
-		(property "LCSC" ""
+		(property "LCSC" "C966144"
 			(at 218.44 104.14 0)
 			(effects
