File: DongleALIVEv2.0.kicad_sch (KiCad schematic)
At the start: 8 parts, among them J1 C-OBD-II-16M, J2 Conn_01x05_Socket, J3 Conn_01x05_Socket

Commit message: Fix tantalum capacitor & JLCPCB codes
Parts:
- J1: LCSC C9900112727 -> (none)
Changed lines of the file:
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@@
 			)
 		)
-		(property "LCSC" "C9900112727"
+		(property "LCSC" ""
 			(at 208.534 97.79 0)
 			(effects

Commit message: Fix CP2102 connection
Changed lines of the file:
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@@
+	(wire
+		(pts
+			(xy 105.41 90.17) (xy 107.95 90.17)
+		)
+		(stroke
+			(width 0)
+			(type default)
+		)
+	)
 	(wire
 		(pts
@@
 	(wire
 		(pts
+			(xy 107.95 90.17) (xy 111.76 93.98)
+		)
+		(stroke
+			(width 0)
+			(type default)
+		)
+	)
+	(wire
+		(pts
 			(xy 109.22 118.11) (xy 101.6 118.11)
 		)
@@
 	(wire
 		(pts
-			(xy 105.41 90.17) (xy 115.824 90.17)
-		)
-		(stroke
-			(width 0)
-			(type default)
-		)
-	)
-	(wire
-		(pts
 			(xy 160.274 118.11) (xy 165.354 118.11)
 		)
@@
 	(wire
 		(pts
+			(xy 107.95 93.98) (xy 111.76 90.17)
+		)
+		(stroke
+			(width 0)
+			(type default)
+		)
+	)
+	(wire
+		(pts
 			(xy 159.004 120.65) (xy 165.354 120.65)
 		)
@@
 	(wire
 		(pts
+			(xy 111.76 93.98) (xy 115.824 93.98)
+		)
+		(stroke
+			(width 0)
+			(type default)
+		)
+	)
+	(wire
+		(pts
+			(xy 111.76 90.17) (xy 115.824 90.17)
+		)
+		(stroke
+			(width 0)
+			(type default)
+		)
+	)
+	(wire
+		(pts
 			(xy 184.658 104.14) (xy 195.834 104.14)
 		)
@@
 	(wire
 		(pts
-			(xy 105.41 93.98) (xy 115.824 93.98)
-		)
-		(stroke
-			(width 0)
-			(type default)
-		)
-	)
-	(wire
-		(pts
 			(xy 184.658 100.33) (xy 195.834 100.33)
+		)
+		(stroke
+			(width 0)
+			(type default)
+		)
+	)
+	(wire
+		(pts
+			(xy 105.41 93.98) (xy 107.95 93.98)
 		)
 		(stroke
@@
 			)
 		)
-		(pin "RXD" output
+		(pin "RXD" input
 			(at 115.824 93.98 180)
 			(effects
@@
 			)
 		)
-		(pin "TXD" input
+		(pin "TXD" output
 			(at 105.41 90.17 0)
 			(effects
