File: DongleALIVEv2.0.kicad_pcb (KiCad board)
At the start: 2 copper layers, 45 x 55 mm, 77 parts, among them J1 C-OBD-II-16M, J2 Conn_01x05_Socket, J3 Conn_01x05_Socket, J4 USB_B_Micro, Q1 IRF5305S, Q2 SS8050-G, Q3 SS8050-G, SW1 SW_Push, SW2 SW_Push, SW3 SW_SPDT_321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

Commit message: Update 01_Specs and Gerber
Connections:
- net /Microcontroller/ESP_RXD renamed /MicroUSB_Port/TXD
- net /Microcontroller/ESP_TXD renamed /MicroUSB_Port/RXD
Changed lines of the file:
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@@
 		(allow_soldermask_bridges_in_footprints no)
 		(pcbplotparams
-			(layerselection 0x00010fc_ffffffff)
+			(layerselection 0x0000000_ffffffff)
 			(plot_on_all_layers_selection 0x0000000_00000000)
 			(disableapertmacros no)
@@
 			(sketchpadsonfab no)
 			(subtractmaskfromsilk no)
-			(outputformat 1)
+			(outputformat 4)
 			(mirror no)
-			(drillshape 0)
+			(drillshape 2)
 			(scaleselection 1)
-			(outputdirectory "02_Gerber&BOM/01_Gerber/00_Drill_Files/")
+			(outputdirectory "01_Specs/02_LayoutPCB/")
 		)
 	)
@@
 	(net 47 "/MicroUSB_Port/DTR")
 	(net 48 "/Microcontroller/TXD0")
-	(net 49 "/Microcontroller/ESP_TXD")
-	(net 50 "/Microcontroller/ESP_RXD")
+	(net 49 "/MicroUSB_Port/RXD")
+	(net 50 "/MicroUSB_Port/TXD")
 	(net 51 "/Microcontroller/CAN_debug")
 	(net 52 "/Microcontroller/BLE_debug")
@@
 			(layers "F.Cu" "F.Paste" "F.Mask")
 			(roundrect_rratio 0.25)
-			(net 49 "/Microcontroller/ESP_TXD")
+			(net 49 "/MicroUSB_Port/RXD")
 			(pinfunction "RXD")
 			(pintype "input")
@@
 			(layers "F.Cu" "F.Paste" "F.Mask")
 			(roundrect_rratio 0.25)
-			(net 50 "/Microcontroller/ESP_RXD")
+			(net 50 "/MicroUSB_Port/TXD")
 			(pinfunction "TXD")
 			(pintype "output")
@@
 			(layers "B.Cu" "B.Paste" "B.Mask")
 			(roundrect_rratio 0.208333)
-			(net 50 "/Microcontroller/ESP_RXD")
+			(net 50 "/MicroUSB_Port/TXD")
 			(pintype "passive")
 		)
@@
 			(layers "B.Cu" "B.Paste" "B.Mask")
 			(roundrect_rratio 0.208333)
-			(net 49 "/Microcontroller/ESP_TXD")
+			(net 49 "/MicroUSB_Port/RXD")
 			(pintype "passive")
 		)
@@
 	)
 	(via
-		(at 136.29 103.61)
+		(at 136.27 103.62)
 		(size 0.7)
 		(drill 0.3)
@@
 	)
 	(segment
-		(start 133.055 98.075)
-		(end 125.705 98.075)
+		(start 132.380105 98.075)
+		(end 127.098 98.075)
 		(width 0.3)
 		(layer "F.Cu")
@@
 	)
 	(segment
-		(start 123.735 100.045)
+		(start 123.73 100.045)
 		(end 123.725 100.045)
 		(width 0.3)
@@
 	)
 	(segment
-		(start 140.425 103.85)
-		(end 138.83 103.85)
+		(start 139.6275 103.85)
+		(end 140.425 103.85)
 		(width 0.3)
 		(layer "F.Cu")
@@
 	)
 	(segment
-		(start 138.83 103.85)
-		(end 133.055 98.075)
+		(start 133.532223 98.552223)
+		(end 138.266082 103.286082)
 		(width 0.3)
 		(layer "F.Cu")
@@
 	)
 	(segment
-		(start 125.705 98.075)
-		(end 123.735 100.045)
+		(start 123.738535 100.041464)
+		(end 124.72 99.06)
+		(width 0.3)
+		(layer "F.Cu")
+		(net 32)
+	)
+	(arc
+		(start 127.098 98.075)
+		(mid 125.811035 98.330993)
+		(end 124.72 99.06)
+		(width 0.3)
+		(layer "F.Cu")
+		(net 32)
+	)
+	(arc
+		(start 133.532223 98.552223)
+		(mid 133.003627 98.199026)
+		(end 132.380105 98.075)
+		(width 0.3)
+		(layer "F.Cu")
+		(net 32)
+	)
+	(arc
+		(start 138.266082 103.286082)
+		(mid 138.890705 103.703442)
+		(end 139.6275 103.85)
+		(width 0.3)
+		(layer "F.Cu")
+		(net 32)
+	)
+	(arc
+		(start 123.738535 100.041464)
+		(mid 123.734619 100.044081)
+		(end 123.73 100.045)
 		(width 0.3)
 		(layer "F.Cu")
@@
 	)
 	(segment
-		(start 132.136989 102.895)
-		(end 132.136989 102.275)
+		(start 132.136989 102.275)
+		(end 132.136989 102.895)
 		(width 0.3)
 		(layer "F.Cu")
@@
 	)
 	(segment
-		(start 132.496989 103.135)
-		(end 132.376989 103.135)
+		(start 132.376989 103.135)
+		(end 132.496989 103.135)
 		(width 0.3)
 		(layer "F.Cu")
@@
 	)
 	(segment
-		(start 140.425 105.12)
-		(end 139.28 105.12)
+		(start 139.8525 105.12)
+		(end 140.425 105.12)
 		(width 0.3)
 		(layer "F.Cu")
@@
 	)
 	(segment
-		(start 139.28 105.12)
-		(end 136.745 102.585)
+		(start 138.875181 104.715181)
+		(end 137.195339 103.035339)
 		(width 0.3)
 		(layer "F.Cu")
@@
 	)
 	(segment
-		(start 131.536989 102.275)
-		(end 131.536989 102.345)
+		(start 131.536989 102.345)
+		(end 131.536989 102.275)
 		(width 0.3)
 		(layer "F.Cu")
@@
 	)
 	(segment
-		(start 131.896989 102.035)
-		(end 131.776989 102.035)
+		(start 131.776989 102.035)
+		(end 131.896989 102.035)
 		(width 0.3)
 		(layer "F.Cu")
@@
 	)
 	(segment
-		(start 136.745 102.585)
+		(start 136.108124 102.585)
 		(end 132.976989 102.585)
 		(width 0.3)
@@
 	)
 	(segment
-		(start 132.736989 102.825)
-		(end 132.736989 102.895)
+		(start 132.736989 102.895)
+		(end 132.736989 102.825)
 		(width 0.3)
 		(layer "F.Cu")
@@
 	)
 	(arc
+		(start 138.875181 104.715181)
+		(mid 139.323578 105.01479)
+		(end 139.8525 105.12)
+		(width 0.3)
+		(layer "F.Cu")
+		(net 33)
+	)
+	(arc
 		(start 132.136989 102.275)
 		(mid 132.066695 102.105294)
@@
 	)
 	(arc
-		(start 132.376989 103.135)
+		(start 132.136989 102.895)
 		(mid 132.207283 103.064706)
-		(end 132.136989 102.895)
+		(end 132.376989 103.135)
 		(width 0.3)
 		(layer "F.Cu")
@@
 	)
 	(arc
+		(start 137.195339 103.035339)
+		(mid 136.696521 102.702039)
+		(end 136.108124 102.585)
+		(width 0.3)
+		(layer "F.Cu")
+		(net 33)
+	)
+	(arc
 		(start 131.776989 102.035)
 		(mid 131.607283 102.105294)
@@
 	)
 	(segment
+		(start 132.115 98.885)
+		(end 133.415 100.185)
+		(width 0.3)
+		(layer "F.Cu")
+		(net 50)
+	)
+	(segment
+		(start 128.005 98.885)
+		(end 132.115 98.885)
+		(width 0.3)
+		(layer "F.Cu")
+		(net 50)
+	)
+	(segment
 		(start 127.887094 105.1842)
 		(end 126.46981 105.1842)
@@
 	)
 	(segment
-		(start 131.835 98.605)
-		(end 133.415 100.185)
-		(width 0.3)
-		(layer "F.Cu")
-		(net 50)
-	)
-	(segment
 		(start 136.7 111.47)
 		(end 136.05 111.47)
@@
 	)
 	(segment
-		(start 128.295 105.592106)
-		(end 127.941447 105.238553)
+		(start 125.805 101.085)
+		(end 128.005 98.885)
 		(width 0.3)
 		(layer "F.Cu")
@@
 	)
 	(segment
-		(start 128.285 98.605)
-		(end 131.835 98.605)
+		(start 128.295 105.592106)
+		(end 127.941447 105.238553)
 		(width 0.3)
 		(layer "F.Cu")
@@
 		(width 0.3)
 		(layer "F.Cu")
-		(net 50)
-	)
-	(segment
-		(start 125.805 101.085)
-		(end 128.285 98.605)
-		(width 0.3)
-		(layer "F.Cu")
